File: hs-64-spi-3d.brd (EAGLE design)
At the start: 19.3 x 18.8 mm, 30 parts, among them J1 DF40C-70DP-0.4V(51), J2 A79622-001, U1 RHD2064_BGA, U2 BNO055, U3 TLV70725

Commit message: Decreased I2C pull-up resistors to 2k.
Parts:
- R7, R8: value 2.2k -> 2k
Changed lines of the file:
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@@
 <attribute name="VALUE" x="3.9998" y="-3.6238" size="1.016" layer="27" font="vector" ratio="18" rot="R180"/>
 </element>
-<element name="R7" library="jonnew" package="0201T" value="2.2k" x="2.4638" y="-0.2413" smashed="yes" rot="R90">
+<element name="R7" library="jonnew" package="0201T" value="2k" x="2.4638" y="-0.2413" smashed="yes" rot="R90">
 <attribute name="NAME" x="2.7178" y="-2.2225" size="0.8128" layer="25" font="vector" ratio="18" rot="R90"/>
 <attribute name="VALUE" x="4.0386" y="-1.4351" size="1.016" layer="27" font="vector" ratio="18" rot="R90"/>
 </element>
-<element name="R8" library="jonnew" package="0201T" value="2.2k" x="3.1623" y="-0.2413" smashed="yes" rot="R90">
+<element name="R8" library="jonnew" package="0201T" value="2k" x="3.1623" y="-0.2413" smashed="yes" rot="R90">
 <attribute name="NAME" x="3.6195" y="-2.2225" size="0.8128" layer="25" font="vector" ratio="19" rot="R90"/>
 <attribute name="VALUE" x="4.7371" y="-1.4351" size="1.016" layer="27" font="vector" ratio="18" rot="R90"/>

Commit message: Connection between REF to GND is now done by default.
Parts:
- R1: value DNP -> 0
Changed lines of the file:
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@@
 <attribute name="NAME" x="-1.1204" y="1.8161" size="0.8128" layer="25" font="vector" ratio="19"/>
 </element>
-<element name="R1" library="jonnew" package="0603" value="DNP" x="-4.0844" y="3.946" smashed="yes">
+<element name="R1" library="jonnew" package="0603" value="0" x="-4.0844" y="3.946" smashed="yes">
 <attribute name="DK" value="PxxxxHTR-ND" x="-4.0844" y="3.946" size="1.778" layer="27" display="off"/>
 <attribute name="MN" value="Panasonic" x="-4.0844" y="3.946" size="1.778" layer="27" display="off"/>

Commit message: Corrected C4 and C7 values to 4.7uF.
Parts:
- C4: value 1uF -> 4.7uF
- C7: value 1u -> 4.7u
Changed lines of the file:
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@@
 <attribute name="NAME" x="-4.718725" y="2.162" size="0.8128" layer="25" font="vector" ratio="19"/>
 </element>
-<element name="C7" library="jonnew" package="0402" value="1u" x="-3.9544" y="-0.7464" smashed="yes" rot="R180">
+<element name="C7" library="jonnew" package="0402" value="4.7u" x="-3.9544" y="-0.7464" smashed="yes" rot="R180">
 <attribute name="NAME" x="-4.4912" y="-0.0298" size="0.8128" layer="25" font="vector" ratio="19"/>
 </element>
@@
 </element>
 <element name="U3" library="jonnew" package="X2SON" value="TLV70725" x="4.5346" y="-5.9412" smashed="yes"/>
-<element name="C4" library="jonnew" package="0402T" value="1uF" x="4.8888" y="-7.009" smashed="yes" rot="R180">
+<element name="C4" library="jonnew" package="0402T" value="4.7uF" x="4.8888" y="-7.009" smashed="yes" rot="R180">
 <attribute name="PARTNO" value="CL05A105KO5NNNC" x="4.8888" y="-8.009" size="1.778" layer="27" rot="R180" display="off"/>
 <attribute name="VALUE" x="6.1588" y="-5.431" size="1.016" layer="27" font="vector" ratio="18" rot="R180"/>

Commit message: Updated Hirose (J1) schematic.
Connections:
- removed net ISTIM: J1.1
- removed net LED-1: J1.34
- removed net LED-2: J1.35
Changed lines of the file:
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@@
 </elements>
 <signals>
-<signal name="LED-2">
-<contactref element="J1" pad="35"/>
-</signal>
 <signal name="VCOAX">
 <contactref element="J1" pad="36"/>
@@
 <contactref element="U1" pad="A9"/>
 <wire x1="0" y1="-0.585" x2="0" y2="-2" width="0.09" layer="16"/>
-</signal>
-<signal name="LED-1">
-<contactref element="J1" pad="34"/>
 </signal>
 <signal name="REF">
@@
 <wire x1="-6.6422" y1="-4.7116" x2="-6.1596" y2="-4.7116" width="0.2032" layer="16"/>
 </signal>
-<signal name="ISTIM">
-<contactref element="J1" pad="1"/>
-</signal>
 <signal name="RESV(VCCIO)">
